File: docs/kicad/lcd_connector/lcd_connector.kicad_pcb (KiCad board)
At the start: 2 copper layers, 17.8 x 38.1 mm, 19 parts, among them J1 5V, J2 T_CS, J3 CLK, J4 MISO, J5 DC, J6 CS, J7 MOSI, J8 GND, M1 TFT_ILI9341

Commit message: continuing work on TE3 kicad designs
Parts:
- M1: footprint cnc3018-PCB:my14Pin -> 0_my_footprints:myPinSocket_1x14
- R1, R2: footprint cnc3018-PCB:myResistor -> 0_my_footprints:myResistor
- moved M1 7.62 mm to (15.2, -2.54), turned to 180 degrees
