File: docs/kicad/mother_board/mother_board.sch (KiCad schematic (older format))
At the start: 13 parts

Commit message: tested prototype rotary board
Parts:
- added R? (x3): 1K, symbol Device:R
Connections:
- wire segments 4 -> 8
Changed lines of the file:
@@
 L Connector_Generic:Conn_01x08 J?
 U 1 1 679456F8
-P 6300 1250
-F 0 "J?" V 6400 850 50  0000 L CNN
-F 1 "TE_DISPLAY" V 6400 1200 50  0000 L CNN
-F 2 "" H 6300 1250 50  0001 C CNN
-F 3 "~" H 6300 1250 50  0001 C CNN
-	1    6300 1250
+P 6200 1250
+F 0 "J?" V 6300 850 50  0000 L CNN
+F 1 "TE_DISPLAY" V 6300 1200 50  0000 L CNN
+F 2 "" H 6200 1250 50  0001 C CNN
+F 3 "~" H 6200 1250 50  0001 C CNN
+	1    6200 1250
 	0    -1   -1   0
 $EndComp
@@
 L power:+5V #PWR?
 U 1 1 6797CEDB
-P 6000 1450
-F 0 "#PWR?" H 6000 1300 50  0001 C CNN
-F 1 "+5V" V 6000 1550 50  0000 L CNN
-F 2 "" H 6000 1450 50  0001 C CNN
-F 3 "" H 6000 1450 50  0001 C CNN
-	1    6000 1450
+P 5900 1450
+F 0 "#PWR?" H 5900 1300 50  0001 C CNN
+F 1 "+5V" V 5900 1550 50  0000 L CNN
+F 2 "" H 5900 1450 50  0001 C CNN
+F 3 "" H 5900 1450 50  0001 C CNN
+	1    5900 1450
 	-1   0    0    1
 $EndComp
@@
 L power:GND #PWR?
 U 1 1 6797D5D1
-P 6700 1450
-F 0 "#PWR?" H 6700 1200 50  0001 C CNN
-F 1 "GND" V 6700 1150 50  0000 L CNN
-F 2 "" H 6700 1450 50  0001 C CNN
-F 3 "" H 6700 1450 50  0001 C CNN
-	1    6700 1450
-	1    0    0    -1
-$EndComp
+P 6600 1450
+F 0 "#PWR?" H 6600 1200 50  0001 C CNN
+F 1 "GND" V 6600 1150 50  0000 L CNN
+F 2 "" H 6600 1450 50  0001 C CNN
+F 3 "" H 6600 1450 50  0001 C CNN
+	1    6600 1450
+	1    0    0    -1
+$EndComp
+Text GLabel 6000 1450 3    50   Input ~ 0
+T41_T_CS
 Text GLabel 6100 1450 3    50   Input ~ 0
-T41_T_CS
+T41_SCLK
 Text GLabel 6200 1450 3    50   Input ~ 0
-T41_SCLK
+T41_MISO
 Text GLabel 6300 1450 3    50   Input ~ 0
-T41_MISO
+T41_LCD_DC
 Text GLabel 6400 1450 3    50   Input ~ 0
-T41_LCD_DC
+T41_LCD_CS
 Text GLabel 6500 1450 3    50   Input ~ 0
-T41_LCD_CS
-Text GLabel 6600 1450 3    50   Input ~ 0
 T41_MOSI
 $Comp
@@
 Text GLabel 11050 3250 1    50   Input ~ 0
 RPI_MOSI
-Text Notes 6100 1100 0    50   ~ 0
+Text Notes 6000 1100 0    50   ~ 0
 ILI9488_T3
 Text GLabel 5150 5100 3    50   Input ~ 0
@@
 U 1 1 64CCBE5B
 P 4500 6500
-F 0 "R?" H 4570 6546 50  0000 L CNN
+F 0 "R?" V 4600 6450 50  0000 L CNN
 F 1 "220" V 4500 6500 50  0000 C CNN
 F 2 "" V 4430 6500 50  0001 C CNN
@@
 	1    0    0    -1
 $EndComp
-Text GLabel 4500 6800 0    50   Input ~ 0
+Text GLabel 4200 6800 0    50   Input ~ 0
 PI_REBOOT
 Wire Wire Line
@@
 Text GLabel 5450 3050 1    50   Input ~ 0
 RPI_READY
+Text GLabel 6150 6700 1    50   Input ~ 0
+T41_SCL
+Text GLabel 6050 6700 1    50   Input ~ 0
+T41_SDA
+$Comp
+L Device:R R?
+U 1 1 67964E23
+P 6050 6850
+F 0 "R?" H 6100 6850 50  0000 L CNN
+F 1 "1K" V 6050 6850 50  0000 C CNN
+F 2 "" V 5980 6850 50  0001 C CNN
+F 3 "~" H 6050 6850 50  0001 C CNN
+	1    6050 6850
+	-1   0    0    1
+$EndComp
+$Comp
+L Device:R R?
+U 1 1 67965E12
+P 6150 6850
+F 0 "R?" H 6000 6850 50  0000 L CNN
+F 1 "1K" V 6150 6850 50  0000 C CNN
+F 2 "" V 6080 6850 50  0001 C CNN
+F 3 "~" H 6150 6850 50  0001 C CNN
+	1    6150 6850
+	-1   0    0    1
+$EndComp
+$Comp
+L power:GND #PWR?
+U 1 1 67968FB3
+P 6100 7100
+F 0 "#PWR?" H 6100 6850 50  0001 C CNN
+F 1 "GND" H 6105 6927 50  0000 C CNN
+F 2 "" H 6100 7100 50  0001 C CNN
+F 3 "" H 6100 7100 50  0001 C CNN
+	1    6100 7100
+	1    0    0    -1
+$EndComp
+Wire Wire Line
+	6050 7000 6050 7100
+Wire Wire Line
+	6050 7100 6100 7100
+Wire Wire Line
+	6150 7000 6150 7100
+Wire Wire Line
+	6150 7100 6100 7100
+Connection ~ 6100 7100
+$Comp
+L Device:R R?
+U 1 1 6796F63B
+P 4350 6800
+F 0 "R?" V 4450 6750 50  0000 L CNN
+F 1 "1K" V 4350 6800 50  0000 C CNN
+F 2 "" V 4280 6800 50  0001 C CNN
+F 3 "~" H 4350 6800 50  0001 C CNN
+	1    4350 6800
+	0    -1   -1   0
+$EndComp
 $EndSCHEMATC

Commit message: built row_board_prototype pcb; added te3_leds (with BC547 level up shifter) and prep for te3_buttons (with 74HC595 polling)
Parts:
- added Q?: BC547, Package_TO_SOT_THT:TO-92_Inline, symbol Transistor_BJT:BC547
- added R?: 6.8K, symbol Device:R
- added R?: 2.2K, symbol Device:R
- added R?: 4.7K, symbol Device:R
- added R?: 10K, symbol Device:R
Connections:
- net labels added: BTN_SENSE_3V, BTN_SENSE_5V, LED_DIN_3V, LED_DIN_5V, T41_5V, T41_RX1, T41_TX1
- net labels removed: BTN_SENSE, LED_DIN, T41_RX5, T41_TX5
- wire segments 8 -> 15
Other:
- note added: "BTN_SENSE goes thru\n5V->3.3V voltage divider"
- note added: "Rotary mcp23017 needs\n1K pullups on SDA & SCL"
- note added: "WS2812b's need\n3.3V->5V level shifter"

Commit message: implemented & tested 2nd row_board prototype 595 buttons; switch to 3.3V row_boards; got rid of 1st row board prototype kicad; ready to start designing motherboard
Parts:
- removed Q?: BC547, Package_TO_SOT_THT:TO-92_Inline, symbol Transistor_BJT:BC547
- removed R?: 6.8K, symbol Device:R
- removed R?: 2.2K, symbol Device:R
- removed R?: 4.7K, symbol Device:R
- removed R?: 10K, symbol Device:R
Connections:
- net labels added: BTN_SENSE, LED_DIN
- net labels removed: BTN_SENSE_3V, BTN_SENSE_5V, LED_DIN_3V, LED_DIN_5V
- wire segments 15 -> 8
Other:
- note removed: "BTN_SENSE goes thru\n5V->3.3V voltage divider"
- note removed: "WS2812b's need\n3.3V->5V level shifter"

Commit message: mother_board schematic comments only
Connections:
- wire segments 8 -> 9
Other:
- note added: "T41 standard SPI SCK is same as ONBOARD_LED.\nI am using a different pin for the display SCLK\non the other side of the board near MISO/MOSI\n"
- note removed: "T41 standard SPI SCK\nconflicts with ONBOARD_LED.\nI will start by leaving it attached\nand using a different pin for\nthe alive led, but it would probably\nbe better on the other side of the\nboard near mosi and CS\n"

Commit message: continuing work on TE3 kicad designs
Parts:
- removed J?: I2S_TXB, symbol Connector_Generic:Conn_01x01
- removed J?: RPI_RUN, symbol Connector_Generic:Conn_01x01
- added J10: rPi_5V, 0_my_footprints:myJSTx02, symbol Connector_Generic:Conn_01x02
- added J11: PEDALS, 0_my_footprints:myJSTx06, symbol Connector_Generic:Conn_01x06
- added J6: I2S_TXB, 0_my_footprints:myJSTx02, symbol Connector_Generic:Conn_01x02
- added J7: RPI_RUN, 0_my_footprints:myJSTx02, symbol Connector_Generic:Conn_01x02
- J1: renamed from J?; footprint (none) -> 0_my_footprints:myJSTx04
- J2: renamed from J?; footprint (none) -> 0_my_footprints:myJSTx06
- J3: renamed from J?; footprint (none) -> 0_my_footprints:myJSTx05
- J4, J5, J8: renamed from J?; footprint (none) -> 0_my_footprints:myJSTx08
- J9: renamed from J?; footprint (none) -> 0_my_footprints2:rpi_zero_2w
- Q1: renamed from Q?; footprint Package_TO_SOT_THT:TO-92_Inline -> 0_my_footprints:myTransistor
- R1, R2, R3, R4: renamed from R?; footprint (none) -> 0_my_footprints:myResistor
- U1: renamed from U?; footprint (none) -> 0_my_teensy:teensy41
- U2: renamed from U?; footprint (none) -> 0_my_teensy:revDTeensy4Stack
Connections:
- net labels added: LED_AUDIO_BUSY, LED_RPI_BUSY, LED_T3_BUSY, PEDAL1, PEDAL2, PEDAL3, PEDAL4
- net labels removed: LED_AUDIO_ALIVE, LED_T3_ALIVE, T41_SCLK?

Commit message: YAY!  Ready to start designing actual mother_board and USBC_connector boards, to move on to 3D printing stuff
Parts:
- removed J1: DBG_SERIAL, 0_my_footprints:myJSTx04, symbol Connector_Generic:Conn_01x04
- removed J11: PEDALS, 0_my_footprints:myJSTx06, symbol Connector_Generic:Conn_01x06
- removed J5: EXT_LEDS, 0_my_footprints:myJSTx08, symbol Connector_Generic:Conn_01x08
- removed U2: teensyAudioRevD, 0_my_teensy:revDTeensy4Stack, symbol 0_my_teensy:teensyAudioRevD
- added C?: 47uf, symbol Device:CP
- added C?: 100uf, symbol Device:CP
- added D? (x3): red, symbol Device:LED_Small
- added D?: green, symbol Device:LED_Small
- added D?: blue, symbol Device:LED_Small
- added D? (x2): yellow, symbol Device:LED_Small
- added J?: PEDAL1, symbol 0_my_symbols:QuarterInchJack1
- added J?: PEDAL2, symbol 0_my_symbols:QuarterInchJack1
- added J?: PEDAL3, symbol 0_my_symbols:QuarterInchJack1
- added J?: PEDAL4, symbol 0_my_symbols:QuarterInchJack1
- added J?: EigthInchJack1, symbol 0_my_symbols:EigthInchJack1
- added J?: GUITAR_IN, symbol 0_my_symbols:QuarterInchJack1
- added J?: LINE_OUT, symbol 0_my_symbols:RCA2_PCB
- added R? (x5): 10K, 0_my_footprints:myResistor, symbol Device:R
- added R? (x7): 220, 0_my_footprints:myResistor, symbol Device:R
- added R?: 100, 0_my_footprints:myResistor, symbol Device:R
- added U?: teensyAudioRevD_WithAudio, symbol 0_my_teensy:teensyAudioRevD_WithAudio
Connections:
- net labels added: LINE_IN_L, LINE_IN_R, LINE_OUT_L, LINE_OUT_R
- net labels removed: T41_5V
- wire segments 9 -> 64
Other:
- note added: "*might* allow for a MIC in 1/8th in jack via \npins on audio shield"
- note added: "Note: NEED TE3 OPTION/CONFIG \nto use MONO LINE_IN_L (tip) for input.\n"
- note removed: "FTDI USB Serial"
- note removed: "T41 standard SPI SCK is same as ONBOARD_LED.\nI am using a different pin for the display SCLK\non the other side of the board near MISO/MOSI\n"

Commit message: design TE3 motherboard
Parts:
- removed D? (x3): red, symbol Device:LED_Small
- removed D?: green, symbol Device:LED_Small
- removed D?: blue, symbol Device:LED_Small
- removed D? (x2): yellow, symbol Device:LED_Small
- removed R? (x6): 220, 0_my_footprints:myResistor, symbol Device:R
- removed R?: 100, 0_my_footprints:myResistor, symbol Device:R
- added J16: LEDS, 0_my_footprints:myJSTx08, symbol Connector_Generic:Conn_01x08
- added R11: 10K, 0_my_footprints:myResistor, symbol Device:R
- C1: renamed from C?; footprint (none) -> 0_my_footprints:CP_my100uf
- C2: renamed from C?; footprint (none) -> 0_my_footprints:CP_my10uf
- J10, J11, J12, J13, J14: renamed from J?; footprint (none) -> 0_my_footprints2:QuarterInchJack1
- J15: renamed from J?; footprint (none) -> 0_my_footprints2:RCA2_PCB
- J9: renamed from J?; footprint (none) -> 0_my_footprints2:EigthInchJack1
- U1: renamed from U?; footprint (none) -> 0_my_teensy:audioShieldRevD_audioPinsStack
- gave numbers to parts that had none: 6
- renumbered J2 to J1, J3 to J2, J4 to J3, J8 to J4, J10 to J5, J7 to J6, J9 to J7, J6 to J8, R4 to R3, R3 to R4, U1 to U2
Connections:
- wire segments 64 -> 46
Other:
- note added: "Note the LED_RPI_BUSY is not implemented yet.\nThe other bold pins depend on #define LOOPER3\nin the circle/Rules.mk makefile to be used in the\n_prh audio and system libraries."
- note added: "Note: NEED TE3 OPTION/CONFIG \nto use MONO LINE_IN_L/R (ring/tip) for input.\n"
- note removed: "Note: NEED TE3 OPTION/CONFIG \nto use MONO LINE_IN_L (tip) for input.\n"

Commit message: kicad changes to support actual Fusion 360 TE3 design efforts - created rotary board PCB
Changed lines of the file:
@@
 F 3 "~" H 3000 1450 50  0001 C CNN
 	1    3000 1450
-	0    -1   -1   0
+	0    1    -1   0
 $EndComp
 $Comp
@@
 	1    0    0    -1
 $EndComp
+Text GLabel 3200 1650 3    50   Input ~ 0
+T41_SCL
+Text GLabel 3100 1650 3    50   Input ~ 0
+T41_SDA
 Text GLabel 2900 1650 3    50   Input ~ 0
-T41_SCL
-Text GLabel 3000 1650 3    50   Input ~ 0
-T41_SDA
-Text GLabel 3100 1650 3    50   Input ~ 0
 ROT_INT
 $Comp
@@
 Text GLabel 2500 3350 1    50   Input ~ 0
 T41_3V3
-Text GLabel 3200 1650 3    50   Input ~ 0
+Text GLabel 3000 1650 3    50   Input ~ 0
 T41_3V3
 Text GLabel 3300 3350 1    50   Input ~ 0
