File: docs/kicad/mother_board/mother_board.sch (KiCad schematic (older format))
At the start: 32 parts, among them J1 ROW_BOARDS, J10 PEDAL1, J11 PEDAL2, J12 PEDAL3, J13 PEDAL4, J14 GUITAR_IN, J15 LINE_OUT, J16 LEDS, J2 ROTARIES, J3 TE_DISPLAY, J4 RPI_DISPLAY, J5 rPi_5V, J6 RPI_RUN, J7 rpi_connector, J8 I2S_TXB, J9 EigthInchJack1, Q1 BC547, U1 teensyAudioRevD_WithAudio, U2 myTeensy4.1

Commit message: cutting actual TE3 milled circuit boards
Changed lines of the file:
@@
 Text GLabel 3400 5400 3    50   Input ~ 0
 T41_LCD_CS
-Text GLabel 3200 5400 3    50   Input ~ 0
+Text GLabel 2700 5400 3    50   Input ~ 0
 T41_T_CS
 Text GLabel 2800 5400 3    50   Input ~ 0

Commit message: final initial TE3 PCBS - updated LED board green resistor to 1K - changed TE3 display SCLK to pin13 as it is required for hardware SPI0 - changed nomenclature of rotary board to ROT0..ROT4 and corrected order to match named rotary 1..4
Changed lines of the file:
@@
 Text Notes 5400 1300 0    50   ~ 0
 ILI9488_T3
-Text GLabel 3100 5400 3    50   Input ~ 0
+Text GLabel 3600 3350 1    50   Input ~ 0
 T41_SCLK
 Text GLabel 3600 5400 3    50   Input ~ 0

Commit message: Fixed problems discovered after milling 1st test mother_board. - effing had I2S BCLK and FCLK going to wrong pins on teensy4.0!! - connector for revD audio pins was off by 1.5mm - separated rPI and teensy 5V rails - needed to use SCLK=pin13 on teensy4.1 for display deleted the old plot files
Connections:
- net labels added: RPI_5V
Other:
- note added: "I2S BCLK and FCLK were WRONG in initial \nbuilt test mother_board, off by one pin to the left,\nGRRRR. with BCLK going to digital pin 22,\nand FCLK going to the BCLK pin!!! They\nhave now been corrected in the schematic\nand PCB which needs to be remade."
- note added: "RPI_5V is separated from teensies +5V.\nThe teensies get their power from the USB hub\nwhich has caps for each plug. The RPI also gets\npower from the hub 5V rail but has its own cap\nand allows for a inline power switch so that it will be \npossible to plug the hub into the laptop/ipad without \nnecessarily powering up the rPI (which draws 1A+)."
- note added: "The bold pins are differfent in Looper3 than previous\nLooper2. They depend on #define LOOPER3\nin the circle/Rules.mk makefile to be used in the\n_prh audio and system libraries."
- note added: "The teensy 5V's are tied together so that both\nwill run if the 4.1 is plugged directly into the laptop."
- note removed: "Note the LED_RPI_BUSY is not implemented yet.\nThe other bold pins depend on #define LOOPER3\nin the circle/Rules.mk makefile to be used in the\n_prh audio and system libraries."

Commit message: found, documented, and fixed test PCB problems with I2S_IXR, LINE_IN_R, GND, and LINE_OUT_R traces (bad schematic and bad kicad symbols)
Other:
- note added: "Built card had I2S_RXB hooked up wrong to gpio5 \nBuilt card, schematic and PCB design modified to\ncorrect pin, gpio6\n"
- note added: "Carnival of errors. Built card had incorrect\nsymbol, with the audio pins showing:\n29 - LINE_IN_L\n30 - GND\n31 - LINE_IN_R\n32 - LINE_OUT_R\n33 - LINE_OUT_L\nThe footprint, built board, schematic\nand PCB design have been fixed as\nshown here.\n\n"
Changed lines of the file:
@@
 Text GLabel 9500 4350 1    50   Input ~ 0
 LINE_OUT_L
-Text GLabel 9400 4350 1    50   Input ~ 0
+Text GLabel 9300 4350 1    50   Input ~ 0
 LINE_OUT_R
 $Comp
@@
 Text GLabel 8200 4000 1    50   Input ~ 0
 I2S_FCLK
-Text GLabel 8200 5450 3    50   Input ~ 0
+Text GLabel 8300 5450 3    50   Input ~ 0
 I2S_RXB
 Text GLabel 9650 5300 2    50   Input ~ 0
@@
 	0    1    -1   0
 $EndComp
-Text GLabel 9300 4350 1    50   Input ~ 0
-LINE_IN_R
-$Comp
-L 0_my_teensy:teensyAudioRevD_WithAudio U1
-U 1 1 67B4E93C
-P 8150 4700
-F 0 "U1" H 7550 4700 60  0000 L CNN
-F 1 "teensyAudioRevD_WithAudio" H 7750 4700 60  0000 L CNN
-F 2 "0_my_teensy:audioShieldRevD_audioPinsStack" V 9100 4650 60  0001 C CNN
-F 3 "" V 9100 4650 60  0000 C CNN
-	1    8150 4700
-	1    0    0    -1
-$EndComp
-$Comp
-L power:GND #PWR020
-U 1 1 67B9218D
-P 9200 4350
-F 0 "#PWR020" H 9200 4100 50  0001 C CNN
-F 1 "GND" V 9200 4050 50  0000 L CNN
-F 2 "" H 9200 4350 50  0001 C CNN
-F 3 "" H 9200 4350 50  0001 C CNN
-	1    9200 4350
-	-1   0    0    1
-$EndComp
 Connection ~ 12400 8750
 Wire Wire Line
@@
 Text GLabel 13500 5200 3    50   Input ~ 0
 RPI_5V
+Text Notes 8200 6350 0    50   ~ 0
+Built card had I2S_RXB hooked up wrong to gpio5 \nBuilt card, schematic and PCB design modified to\ncorrect pin, gpio6\n
+Text Notes 9650 4100 0    50   ~ 0
+Carnival of errors.  Built card had incorrect\nsymbol, with the audio pins showing:\n29 - LINE_IN_L\n30 - GND\n31 - LINE_IN_R\n32 - LINE_OUT_R\n33 - LINE_OUT_L\nThe footprint, built board, schematic\nand PCB design have been fixed as\nshown here.\n\n
+Text GLabel 9200 4350 1    50   Input ~ 0
+LINE_IN_R
+$Comp
+L power:GND #PWR020
+U 1 1 67B9218D
+P 9400 4350
+F 0 "#PWR020" H 9400 4100 50  0001 C CNN
+F 1 "GND" V 9400 4050 50  0000 L CNN
+F 2 "" H 9400 4350 50  0001 C CNN
+F 3 "" H 9400 4350 50  0001 C CNN
+	1    9400 4350
+	-1   0    0    1
+$EndComp
+$Comp
+L 0_my_teensy:teensyAudioRevD_WithAudio U1
+U 1 1 67B4E93C
+P 8150 4700
+F 0 "U1" H 7550 4700 60  0000 L CNN
+F 1 "teensyAudioRevD_WithAudio" H 7750 4700 60  0000 L CNN
+F 2 "0_my_teensy:audioShieldRevD_audioPinsStack" V 9100 4650 60  0001 C CNN
+F 3 "" V 9100 4650 60  0000 C CNN
+	1    8150 4700
+	1    0    0    -1
+$EndComp
 $EndSCHEMATC

Commit message: produced and submitted mother_board and row_board to PCBWay for production
Parts:
- removed R10, R6, R7, R8, R9: 10K, 0_my_footprints:myResistor, symbol Device:R
- J15: footprint 0_my_footprints2:RCA2_PCB -> 0_my_footprints2:RCA2_PCB_milled
- J7: footprint 0_my_footprints2:rpi_zero_2w -> 0_my_footprints2:rpi_zero_2w_for_TE3
Connections:
- wire segments 46 -> 36
Changed lines of the file:
@@
 F 0 "J7" H 12200 4500 50  0000 L CNN
 F 1 "rpi_connector" H 12350 4500 50  0000 L CNN
-F 2 "0_my_footprints2:rpi_zero_2w" H 12450 4400 50  0001 C CNN
+F 2 "0_my_footprints2:rpi_zero_2w_for_TE3" H 12450 4400 50  0001 C CNN
 F 3 "" H 12450 4400 50  0001 C CNN
 	1    12550 4500
@@
 $EndComp
 $Comp
-L Device:R R6
-U 1 1 67ACD401
-P 3750 8100
-F 0 "R6" V 3850 8050 50  0000 L CNN
-F 1 "10K" V 3750 8100 50  0000 C CNN
-F 2 "0_my_footprints:myResistor" V 3680 8100 50  0001 C CNN
-F 3 "~" H 3750 8100 50  0001 C CNN
-	1    3750 8100
-	-1   0    0    1
-$EndComp
-$Comp
-L Device:R R7
-U 1 1 67ACDF8A
-P 5050 8100
-F 0 "R7" V 5150 8050 50  0000 L CNN
-F 1 "10K" V 5050 8100 50  0000 C CNN
-F 2 "0_my_footprints:myResistor" V 4980 8100 50  0001 C CNN
-F 3 "~" H 5050 8100 50  0001 C CNN
-	1    5050 8100
-	-1   0    0    1
-$EndComp
-$Comp
-L Device:R R8
-U 1 1 67ACE349
-P 6300 8100
-F 0 "R8" V 6400 8050 50  0000 L CNN
-F 1 "10K" V 6300 8100 50  0000 C CNN
-F 2 "0_my_footprints:myResistor" V 6230 8100 50  0001 C CNN
-F 3 "~" H 6300 8100 50  0001 C CNN
-	1    6300 8100
-	-1   0    0    1
-$EndComp
-$Comp
-L Device:R R9
-U 1 1 67ACFA4C
-P 7550 8100
-F 0 "R9" V 7650 8050 50  0000 L CNN
-F 1 "10K" V 7550 8100 50  0000 C CNN
-F 2 "0_my_footprints:myResistor" V 7480 8100 50  0001 C CNN
-F 3 "~" H 7550 8100 50  0001 C CNN
-	1    7550 8100
-	-1   0    0    1
-$EndComp
-$Comp
 L 0_my_symbols:EigthInchJack1 J9
 U 1 1 67AFA9BD
@@
 F 0 "J15" V 10500 9250 50  0000 R CNN
 F 1 "LINE_OUT" V 10500 9050 50  0000 R CNN
-F 2 "0_my_footprints2:RCA2_PCB" H 10800 8550 50  0001 C CNN
+F 2 "0_my_footprints2:RCA2_PCB_milled" H 10800 8550 50  0001 C CNN
 F 3 "" H 10800 8550 50  0001 C CNN
 	1    10800 8950
@@
 $EndComp
 Wire Wire Line
-	7550 7800 7550 7950
-Wire Wire Line
 	3000 7800 3500 7800
 Wire Wire Line
 	7300 7800 7300 8250
-Connection ~ 7300 7800
-Wire Wire Line
-	7300 7800 7550 7800
-Wire Wire Line
-	6300 7950 6300 7800
-Connection ~ 6300 7800
-Wire Wire Line
-	6300 7800 7300 7800
 Wire Wire Line
 	6050 7800 6050 8250
 Connection ~ 6050 7800
 Wire Wire Line
-	6050 7800 6300 7800
-Wire Wire Line
-	5050 7950 5050 7800
-Connection ~ 5050 7800
-Wire Wire Line
-	5050 7800 6050 7800
-Wire Wire Line
 	4800 7800 4800 8250
 Connection ~ 4800 7800
 Wire Wire Line
-	4800 7800 5050 7800
-Wire Wire Line
-	3750 7950 3750 7800
-Connection ~ 3750 7800
-Wire Wire Line
-	3750 7800 4800 7800
-Wire Wire Line
 	3500 7800 3500 8250
 Connection ~ 3500 7800
 Wire Wire Line
-	3500 7800 3750 7800
-$Comp
-L Device:R R10
-U 1 1 67A8E02B
-P 9350 8100
-F 0 "R10" V 9450 8050 50  0000 L CNN
-F 1 "10K" V 9350 8100 50  0000 C CNN
-F 2 "0_my_footprints:myResistor" V 9280 8100 50  0001 C CNN
-F 3 "~" H 9350 8100 50  0001 C CNN
-	1    9350 8100
-	-1   0    0    1
-$EndComp
-Wire Wire Line
 	9000 7850 9100 7850
 Wire Wire Line
-	9350 7850 9350 7950
-Wire Wire Line
 	9100 8250 9100 7850
-Connection ~ 9100 7850
-Wire Wire Line
-	9100 7850 9350 7850
 Wire Wire Line
 	12400 8800 12400 8750
@@
 	1    0    0    -1
 $EndComp
+Wire Wire Line
+	3500 7800 4800 7800
+Wire Wire Line
+	4800 7800 6050 7800
+Wire Wire Line
+	6050 7800 7300 7800
 $EndSCHEMATC
