File: docs/kicad/led_board/led_board.kicad_pcb (KiCad board)
At the start: 2 copper layers, 27.9 x 27.9 mm, 19 parts, among them J1 Conn_01x08

Commit message: final initial TE3 PCBS - updated LED board green resistor to 1K - changed TE3 display SCLK to pin13 as it is required for hardware SPI0 - changed nomenclature of rotary board to ROT0..ROT4 and corrected order to match named rotary 1..4
Other:
- board text added: "1K"
- board text removed: "100"
